File: CARGADOR DE BATERIA/CARGADOR DE BATERIA.kicad_pcb (KiCad board)
At the start: 2 copper layers, 49.5 x 24.1 mm, 12 parts, among them P1 out, P2 pwr, U1 TP4056

Commit message: arreglando la tierra
Routing:
- net VCC: track 54.9 -> 57.9 mm
- net /BAT: track 54.6 -> 53.7 mm
Changed lines of the file:
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@@
     (thickness 1.6)
     (drawings 11)
-    (tracks 63)
+    (tracks 69)
     (zones 0)
     (modules 12)
@@
   (gr_line (start 154.94 85.09) (end 105.41 85.09) (angle 90) (layer Edge.Cuts) (width 0.15))
   (gr_line (start 154.94 109.22) (end 154.94 85.09) (angle 90) (layer Edge.Cuts) (width 0.15))
+  (segment (start 139.18946 97.79254) (end 140.96746 97.79254) (width 0.8) (layer F.Cu) (net 1) (status 400000))
+  (segment (start 142.24 93.345) (end 144.145 91.44) (width 0.8) (layer F.Cu) (net 1) (status 800000))
+  (segment (start 142.24 96.52) (end 142.24 93.345) (width 0.8) (layer F.Cu) (net 1))
+  (segment (start 140.96746 97.79254) (end 142.24 96.52) (width 0.8) (layer F.Cu) (net 1))
+  (segment (start 144.145 91.44) (end 144.78 91.44) (width 0.8) (layer F.Cu) (net 1) (status C00000))
   (segment (start 122.43054 105.40746) (end 135.608316 105.40746) (width 0.8) (layer F.Cu) (net 1))
   (segment (start 135.608316 105.40746) (end 136.730662 104.285114) (width 0.8) (layer F.Cu) (net 1))
@@
   (segment (start 144.78 91.44) (end 140.97 91.44) (width 0.8) (layer F.Cu) (net 1))
   (segment (start 140.97 91.44) (end 133.35 91.44) (width 0.8) (layer F.Cu) (net 1))
-  (segment (start 139.18946 97.79254) (end 139.18946 93.22054) (width 0.8) (layer F.Cu) (net 1))
-  (segment (start 139.18946 93.22054) (end 140.97 91.44) (width 0.8) (layer F.Cu) (net 1))
   (segment (start 149.86 91.44) (end 144.78 91.44) (width 0.8) (layer F.Cu) (net 1))
   (segment (start 114.3 88.9) (end 117.910446 88.9) (width 0.25) (layer F.Cu) (net 2))
@@
   (segment (start 118.11 102.91) (end 122.388 102.91) (width 0.25) (layer F.Cu) (net 2))
   (segment (start 122.388 102.91) (end 122.43054 102.86746) (width 0.25) (layer F.Cu) (net 2))
+  (segment (start 109.22 99.06) (end 111.76 99.06) (width 0.8) (layer F.Cu) (net 3) (status 400000))
+  (segment (start 116.84 96.52) (end 118.11 96.52) (width 0.8) (layer F.Cu) (net 3) (status 800000))
+  (segment (start 116.205 95.885) (end 116.84 96.52) (width 0.8) (layer F.Cu) (net 3))
+  (segment (start 113.03 95.885) (end 116.205 95.885) (width 0.8) (layer F.Cu) (net 3))
+  (segment (start 112.395 96.52) (end 113.03 95.885) (width 0.8) (layer F.Cu) (net 3))
+  (segment (start 112.395 98.425) (end 112.395 96.52) (width 0.8) (layer F.Cu) (net 3))
+  (segment (start 111.76 99.06) (end 112.395 98.425) (width 0.8) (layer F.Cu) (net 3))
   (segment (start 109.22 99.06) (end 108.178502 99.06) (width 0.8) (layer F.Cu) (net 3))
   (segment (start 108.178502 99.06) (end 107.052676 100.185826) (width 0.8) (layer F.Cu) (net 3))
@@
   (segment (start 137.562362 107.593651) (end 139.18946 105.966553) (width 0.8) (layer F.Cu) (net 3))
   (segment (start 139.18946 105.966553) (end 139.18946 105.40746) (width 0.8) (layer F.Cu) (net 3))
-  (segment (start 109.22 99.06) (end 109.22 96.52) (width 0.8) (layer F.Cu) (net 3))
-  (segment (start 116.84 95.25) (end 118.11 96.52) (width 0.8) (layer F.Cu) (net 3))
-  (segment (start 110.49 95.25) (end 116.84 95.25) (width 0.8) (layer F.Cu) (net 3))
-  (segment (start 109.22 96.52) (end 110.49 95.25) (width 0.8) (layer F.Cu) (net 3))
   (segment (start 144.78 97.79) (end 144.78 93.98) (width 0.8) (layer F.Cu) (net 4))
   (segment (start 149.86 97.79) (end 149.86 93.98) (width 0.8) (layer F.Cu) (net 5))
